File: pcb.kicad_pcb (KiCad board)
At the start: 2 copper layers, 24 parts, among them SW1 SW_Push, U1 ATmega32U4-AU, Y1 16MHz

Commit message: final
Parts:
- moved C2 24.6 mm to (128.7, 102.8)
- moved C4 11.1 mm to (132.3, 106.5), turned to 90 degrees
- moved C7 7.25 mm to (121.3, 96.9)
- moved C6 4.60 mm to (136.0, 80.6)
- moved C1 3.16 mm to (130.9, 82.8), turned to 0 degrees
- moved R1 2.67 mm to (116.1, 88.0)
- moved R2 2.34 mm to (119.8, 88.0)
Routing:
- net GND: track 0.00 -> 39.4 mm
- net +5V: track 0.00 -> 28.5 mm
- net Net-(R1-Pad1): track 0.00 -> 18.2 mm
- net Net-(R2-Pad1): track 0.00 -> 17.2 mm
- net Net-(C4-Pad1): track 0.00 -> 13.4 mm
- net Net-(C3-Pad1): track 0.00 -> 9.35 mm
- net D+: track 0.00 -> 4.54 mm
- net D-: track 0.00 -> 4.47 mm
Other:
- net class Power added: clearance 0.2, trace_width 0.381, via_dia 0.8, via_drill 0.4
